Commit message: Version3.2

File: urdf/humanoidV3.urdf (robot description, URDF)
Before this commit: robot humanoidV3, 38 links, 37 joints
Links:
- added link sensor1, mass 0.00111; collision mesh filename=meshes/sensor1.stl scale=0.001 0.001 0.001; visual mesh filename=meshes/sensor1.stl scale=0.001 0.001 0.001
- added link sensor2, mass 0.00111; collision mesh filename=meshes/sensor2.stl scale=0.001 0.001 0.001; visual mesh filename=meshes/sensor2.stl scale=0.001 0.001 0.001
- added link sensor3, mass 0.00111; collision mesh filename=meshes/sensor3.stl scale=0.001 0.001 0.001; visual mesh filename=meshes/sensor3.stl scale=0.001 0.001 0.001
- added link sensor4, mass 0.00111; collision mesh filename=meshes/sensor4.stl scale=0.001 0.001 0.001; visual mesh filename=meshes/sensor4.stl scale=0.001 0.001 0.001
- added link sensor5, mass 0.00111; collision mesh filename=meshes/sensor5.stl scale=0.001 0.001 0.001; visual mesh filename=meshes/sensor5.stl scale=0.001 0.001 0.001
- added link sensor6, mass 0.00111; collision mesh filename=meshes/sensor6.stl scale=0.001 0.001 0.001; visual mesh filename=meshes/sensor6.stl scale=0.001 0.001 0.001
- added link sensor7, mass 0.00111; collision mesh filename=meshes/sensor7.stl scale=0.001 0.001 0.001; visual mesh filename=meshes/sensor7.stl scale=0.001 0.001 0.001
Joints:
- removed joint servo10_val
- removed joint servo11_val
- removed joint servo12_val
- removed joint servo13_val
- removed joint servo14_val
- removed joint servo15_val
- removed joint servo16_val
- removed joint servo17_val
- removed joint servo1_val
- removed joint servo2_val
- removed joint servo3_val
- removed joint servo4_val
- removed joint servo5_val
- removed joint servo6_val
- removed joint servo7_val
- removed joint servo8_val
- removed joint servo9_val
- added joint Comp4_Revolute-122: type revolute, parent Comp4, child servo17, origin xyz=0.0 0.0 0.06 rpy=9.860761315262648e-32 -0.0 1.0729844052798728e-32, axis 0.0 9.860761315262648e-32 1.0, limit lower=-1.570796 upper=1.570796 effort=1000000 velocity=1000000
- added joint Comp4_Rigid-145: type fixed, parent Comp4, child sensor7, origin xyz=-0.01 0.0 0.03 rpy=1.0729844052798728e-32 -1.5707963267948966 0
- added joint csmall11_Revolute-117: type revolute, parent csmall11, child servo14, origin xyz=0.0 -0.02475 0.033 rpy=-1.5707963267948966 1.5707963267948966 0, axis 1.8347383247374562e-31 1.9721522630525295e-31 1.0, limit lower=-0.349066 upper=2.792527 effort=1000000 velocity=1000000
- added joint csmall12_Revolute-115: type revolute, parent csmall12, child servo12, origin xyz=0.0 0.02475 0.03300000000000001 rpy=1.5707963267948966 3.0814879110195774e-33 -1.1885773227884292e-31, axis -9.527285330385062e-32 0.0 1.0, limit lower=-1.570796 upper=1.570796 effort=1000000 velocity=1000000
- added joint csmall14_Revolute-124: type revolute, parent csmall14, child servo13, origin xyz=0.0 0.02475 0.03300000000000001 rpy=1.5707963267948966 -1.5707963267948966 0, axis -3.697738713728978e-32 1.9721522630525295e-31 1.0, limit lower=-2.96706 upper=0.174533 effort=1000000 velocity=1000000
- added joint csmall15_Revolute-110: type revolute, parent csmall15, child servo11, origin xyz=0.0 0.02475 0.03300000000000001 rpy=1.5707963267948966 9.860761315262648e-32 5.28375221563461e-32, axis -3.797217091082633e-32 0.0 1.0, limit lower=-1.570796 upper=1.570796 effort=1000000 velocity=1000000
- added joint csmall1_Revolute-87: type revolute, parent csmall1, child servo2, origin xyz=0.0 0.024749999999999998 0.033 rpy=1.5707963267948966 9.860761315262648e-32 1.4739898164836845e-31, axis -7.992343164533666e-32 0.0 1.0, limit lower=-0.872665 upper=0.872665 effort=1000000 velocity=1000000
- added joint csmall2_Revolute-91: type revolute, parent csmall2, child servo4, origin xyz=-0.02475 0.0 0.033 rpy=1.9734305032509502e-31 1.5707963267948966 0, axis 7.888609052210118e-31 5.227728254181639e-31 1.0, limit lower=-1.570796 upper=1.570796 effort=1000000 velocity=1000000
- added joint csmall4_Revolute-96: type revolute, parent csmall4, child servo8, origin xyz=-0.024749999999999998 0.0 0.03300000000000001 rpy=7.992286107048302e-32 1.5707963267948966 0, axis 0.0 2.7962383350627467e-31 1.0, limit lower=-1.570796 upper=1.570796 effort=1000000 velocity=1000000
- added joint csmall6_Revolute-88: type revolute, parent csmall6, child servo1, origin xyz=0.0 0.024749999999999998 0.033 rpy=1.5707963267948966 -4.930380657631324e-32 -1.97324315788137e-31, axis 3.1492006061600383e-32 -3.944304526105059e-31 1.0, limit lower=-0.872665 upper=0.872665 effort=1000000 velocity=1000000
- added joint csmall7_Revolute-100: type revolute, parent csmall7, child servo3, origin xyz=0.024750000000000015 0.0 0.033 rpy=3.141592653589793 1.5707963267948966 0, axis -7.888609052210118e-31 1.6743631100220177e-31 1.0, limit lower=-1.570796 upper=1.570796 effort=1000000 velocity=1000000
- added joint csmall9_Revolute-105: type revolute, parent csmall9, child servo7, origin xyz=0.024749999999999998 0.0 0.03300000000000001 rpy=3.141592653589793 1.5707963267948966 0, axis -3.944304526105059e-31 -1.8538350212600917e-31 1.0, limit lower=-1.570796 upper=1.570796 effort=1000000 velocity=1000000
- added joint servo10_Revolute-98: type revolute, parent servo10, child csmall5, origin xyz=-0.0025 -0.026000000000000002 0.03 rpy=1.5707963267948966 1.5707963267948966 0, axis 2.7286503733033063e-32 -0.0 1.0, limit lower=-1.570796 upper=0.523599 effort=1000000 velocity=1000000
- added joint servo11_Rigid-144: type fixed, parent servo11, child sensor5, origin xyz=0.011750000000000007 0.03527048000000001 0.0260249 rpy=-1.5707963267948966 2.9954761117921433e-62 -1.5707963267948966
- added joint servo12_Rigid-143: type fixed, parent servo12, child sensor6, origin xyz=-0.011749999999999998 0.03527048000000001 0.0260249 rpy=1.5707963267948966 -0.0 -1.5707963267948966
- added joint servo15_Revolute-113: type revolute, parent servo15, child csmall14, origin xyz=0.0025 0.038999999999999986 0.01 rpy=-1.5707963267948966 -1.5707963267948966 0, axis -7.888609052210118e-31 -2.4764777820344067e-31 1.0, limit lower=-2.792527 upper=0.349066 effort=1000000 velocity=1000000
- added joint servo16_Revolute-118: type revolute, parent servo16, child csmall11, origin xyz=0.0025 -0.03899999999999999 0.01 rpy=1.5707963267948966 -1.5707963267948966 0, axis 0.0 -4.8337454333703625e-31 1.0, limit lower=-0.349066 upper=2.792527 effort=1000000 velocity=1000000
- added joint servo1_Rigid-139: type fixed, parent servo1, child sensor1, origin xyz=0.01 -0.01 0.025999999999999995 rpy=1.5707963267948966 -5.702138497759798e-33 -9.860761315262648e-32
- added joint servo2_Rigid-140: type fixed, parent servo2, child sensor2, origin xyz=-0.01 -0.01 0.025999999999999995 rpy=1.5707963267948966 -4.4320160466905134e-32 9.860761315262648e-32
- added joint servo5_Revolute-103: type revolute, parent servo5, child csmall8, origin xyz=0.02655113000000002 -0.07088231999999998 -0.01 rpy=1.5707963267948966 -1.9721522630525295e-31 1.5707963267948966, axis -3.944304526105059e-31 -7.727863396283102e-32 1.0, limit lower=-1.570796 upper=1.570796 effort=1000000 velocity=1000000
- added joint servo5_Rigid-142: type fixed, parent servo5, child sensor3, origin xyz=0.0005511300000000042 -0.06088231999999998 -0.025 rpy=-3.141592653589793 2.500881773550205e-31 4.93211964933386e-62
- added joint servo6_Revolute-94: type revolute, parent servo6, child csmall3, origin xyz=-0.026551129999999996 -0.07088231999999998 -0.01 rpy=-1.5707963267948966 -0.0 1.5707963267948966, axis 0.0 -1.159031063722169e-33 1.0, limit lower=-1.570796 upper=1.570796 effort=1000000 velocity=1000000
- added joint servo6_Rigid-141: type fixed, parent servo6, child sensor4, origin xyz=-0.0005511299999999953 -0.06088231999999998 -0.025 rpy=3.141592653589793 6.518783011447375e-32 -9.860761315262648e-32
- added joint servo9_Revolute-107: type revolute, parent servo9, child csmall10, origin xyz=-0.0025 0.026000000000000002 0.03 rpy=-1.5707963267948966 -1.5707963267948966 0, axis 2.728650373303245e-32 -0.0 1.0, limit lower=-0.523599 upper=1.570796 effort=1000000 velocity=1000000
- joint Comp1_Rigid-92: origin xyz=0.0 0.01046829 0.014202469999999998 rpy=0.0 -0.0 -1.6358743464059394e-31 -> xyz=0.0 0.01046829 0.014202469999999998 rpy=1.9721522630525295e-31 -5.616505753082788e-63 -2.84790675563228e-32
- joint Comp2_Rigid-101: origin xyz=0.0 0.01046829 0.014202469999999998 rpy=3.944304526105059e-31 -9.860761315262648e-32 -1.5531252759231369e-31 -> xyz=0.0 0.01046829 0.014202469999999998 rpy=-3.944304526105059e-31 -0.0 -6.221834973550431e-32
- joint Comp3_Rigid-114: origin xyz=0.055 0.0 0.03 rpy=0.0 3.944304526105059e-31 -1.5707963267948966 -> xyz=0.055 0.0 0.029999999999999964 rpy=-1.1846452909010346e-63 1.9721522630525295e-31 -1.5707963267948966
- joint Comp3_Rigid-119: origin xyz=-0.05499999999999999 0.0 0.03 rpy=0.0 3.944304526105059e-31 -1.5707963267948966 -> xyz=-0.05500000000000001 0.0 0.029999999999999964 rpy=-1.1846452909010346e-63 1.9721522630525295e-31 -1.5707963267948966
- joint Comp3_Rigid-121: origin xyz=0.0 0.0 0.03 rpy=3.944304526105059e-31 -0.0 -2.9824285462269747e-32 -> xyz=0.0 0.0 0.029999999999999964 rpy=1.9721522630525295e-31 1.1846452909010346e-63 -6.006865256272968e-33
- joint base_link_Rigid-108: origin xyz=0.09800000173564674 -0.0009999970614000986 0.29436807577873964 rpy=-3.141592653589793 -1.5707963267948921 0 -> xyz=0.09800000364404338 -0.00099999706139963 0.2943680748627 rpy=-3.1415926535897927 -1.5707963267948928 0
- joint base_link_Rigid-109: origin xyz=0.08750000173564716 -0.0009999970614000986 0.30713552577873926 rpy=-2.1459482208350834e-15 5.377642775528099e-16 1.4131517269391567e-16 -> xyz=0.08750000364404383 -0.0009999970613996235 0.3071355248626996 rpy=-1.2577698011349667e-15 4.2674197509029474e-16 7.021478737325924e-16
- joint base_link_Rigid-99: origin xyz=0.07700000173564747 -0.0009999970614001019 0.29436807577873964 rpy=1.4131517269391505e-16 -1.5707963267948921 0 -> xyz=0.07700000364404411 -0.0009999970613996456 0.2943680748627 rpy=7.021478737325863e-16 -1.5707963267948928 0
- joint csmall10_Rigid-106: origin xyz=0.0 -0.03300000000000001 -0.02475 rpy=1.5707963267948966 4.954121711661801e-32 0.0 -> xyz=0.0 -0.03300000000000001 -0.02475 rpy=1.5707963267948966 2.784067740973774e-31 0.0
- joint csmall3_Rigid-93: origin xyz=-0.03300000000000001 0.0 -0.024749999999999998 rpy=3.141592653589793 1.5707963267948966 0 -> xyz=-0.03300000000000001 0.0 -0.02475 rpy=-3.141592653589793 1.5707963267948966 0
- joint csmall5_Rigid-97: origin xyz=0.0 -0.03300000000000001 -0.02475 rpy=1.5707963267948966 -3.654358718453336e-32 -9.860761315262648e-32 -> xyz=0.0 -0.03300000000000001 -0.02475 rpy=1.5707963267948966 -2.1340054758171858e-32 9.860761315262648e-32
- joint csmall8_Rigid-102: origin xyz=-0.03300000000000001 0.0 -0.024750000000000015 rpy=-4.930380657631324e-32 -1.5707963267948966 0 -> xyz=-0.03300000000000001 0.0 -0.024750000000000015 rpy=-1.9721522630525295e-31 -1.5707963267948966 0
- joint servo13_Rigid-123: origin xyz=-0.0025 0.03 0.026000000000000002 rpy=-1.5707963267948966 3.5141268180324735e-33 0.0 -> xyz=-0.0025 0.029999999999999964 0.026000000000000002 rpy=-1.5707963267948966 -5.184273838280954e-32 0.0
- joint servo14_Rigid-116: origin xyz=0.0025 0.03 0.026000000000000002 rpy=-1.5707963267948966 -2.175320663350183e-32 -1.232595164407831e-32 -> xyz=0.0025 0.029999999999999964 0.026000000000000002 rpy=-1.5707963267948966 3.976044180564392e-31 3.0814879110195774e-33
- joint servo1_Rigid-86: origin xyz=0.01 0.015 0.025999999999999995 rpy=-1.5707963267948966 -1.0586267447530742e-31 0.0 -> xyz=0.01 0.015 0.025999999999999995 rpy=-1.5707963267948966 -5.702138497759798e-33 -9.860761315262648e-32
- joint servo2_Rigid-85: origin xyz=-0.01 0.015 0.025999999999999995 rpy=-1.5707963267948966 1.2948285703496187e-32 5.107198190560144e-63 -> xyz=-0.01 0.015 0.025999999999999995 rpy=-1.5707963267948966 -4.4320160466905134e-32 9.860761315262648e-32
- joint servo3_Rigid-89: origin xyz=-0.01500000000000001 0.01 0.026000000000000016 rpy=3.141592653589793 1.5707963267948966 0 -> xyz=-0.015 0.01 0.026000000000000016 rpy=-3.141592653589793 1.5707963267948966 0
- joint servo4_Rigid-90: origin xyz=-0.01500000000000001 -0.01 0.025999999999999995 rpy=-2.1829489392438793e-62 -1.5707963267948966 0 -> xyz=-0.015 -0.01 0.026000000000000002 rpy=-0.0 -1.5707963267948966 0
- joint servo8_Rigid-95: origin xyz=-0.01 0.015 0.026000000000000002 rpy=-1.5707963267948966 -1.5707963267948966 0 -> xyz=-0.01 0.015 0.025999999999999995 rpy=-1.5707963267948966 -1.5707963267948966 0
